File: H-Bridge-MD.kicad_pcb (KiCad board)
At the start: 2 copper layers, 85 x 50 mm, 68 parts, among them IC1 SI8650AB-B-IS1, IC2 A3921KLPTR-T, IC3 SI8650AB-B-IS1, IC4 A3921KLPTR-T, J1 Conn_01x02, J2 Conn_01x03, J3 Conn_01x05, J4 Conn_01x02, J5 Bus_mechaken_PCIexpress_x16_1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, Q1 NVMFD5C446NT1G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

Commit message: fix
Parts:
- added S2: DIPSW, Package_DIP:DIP-8_W7.62mm, B.Cu at (60.2, 51.1)
- R15, R18: value 3.74k -> 10k
- R16, R19: value 1.2k -> 2.2k
Routing:
- net +3V3: track 119.5 -> 122.4 mm
- net DIP_SW_4: track 7.44 -> 8.18 mm
- net DIP_SW_3: track 8.28 -> 9.02 mm
- net DIP_SW_1: track 9.95 -> 10.7 mm
- net DIP_SW_2: track 8.83 -> 9.58 mm
